Commit message: new commit

File: src/turtlebot3_description/urdf/turtlebot3_waffle.gazebo.xacro (robot description, xacro)
@@ -4,14 +4,16 @@
   <xacro:arg name="camera_visual" default="false"/>
   <xacro:arg name="imu_visual"    default="false"/>
- <xacro:arg name="self_collida"    default="false"/>
+  <xacro:arg name="self_collida"    default="true"/>
   <gazebo reference="base_link">
     <material>Gazebo/DarkGrey</material>
   </gazebo>
 <gazebo reference="bowl_link">
-    <mu1>1</mu1>
-    <mu2>1</mu2>
-    <kp>500000.0</kp>
-    <kd>10.0</kd>
-    <minDepth>0.00000</minDepth>
+    <mu1>0.4</mu1>
+    <mu2>0.4</mu2>
+    <kp>500000.0</kp>
+    <kd>10.0</kd>
+    <minDepth>0.001</minDepth>
+    <material>Gazebo/Grass</material>
+    <selfCollide>true</selfCollide>
     <fdir1>1 0 0</fdir1>
   </gazebo>
@@ -21,12 +23,13 @@
     <kp>500000.0</kp>
     <kd>10.0</kd>
-    <minDepth>0.001</minDepth>
-    <maxVel>0.1</maxVel>
-    <fdir1>1 0 0</fdir1>
-    <material>Gazebo/Green</material>
+    <minDepth>0.00001</minDepth>
+    <maxVel>0.01</maxVel>
+    <fdir1>1 0 0</fdir1>
+    <selfCollide>true</selfCollide>
+    <material>Gazebo/Wood</material>
   </gazebo>-->
   <gazebo reference="wheel_left_link">
-    <mu1>0.1</mu1>
-    <mu2>0.1</mu2>
+    <mu1>1.5</mu1>
+    <mu2>1.5</mu2>
     <kp>500000.0</kp>
     <kd>10.0</kd>
@@ -37,6 +40,6 @@
   </gazebo>
   <gazebo reference="wheel_right_link">
-    <mu1>0.1</mu1>
-    <mu2>0.1</mu2>
+    <mu1>1</mu1>
+    <mu2>1</mu2>
     <kp>500000.0</kp>
     <kd>10.0</kd>
@@ -47,6 +50,6 @@
   </gazebo>
   <gazebo reference="caster_back_right_link">
-    <mu1>0.1</mu1>
-    <mu2>0.1</mu2>
+    <mu1>0.5</mu1>
+    <mu2>0.5</mu2>
     <kp>1000000.0</kp>
     <kd>100.0</kd>
@@ -56,6 +59,6 @@
   </gazebo>
   <gazebo reference="caster_back_left_link">
-    <mu1>0.1</mu1>
-    <mu2>0.1</mu2>
+    <mu1>0.5</mu1>
+    <mu2>0.5</mu2>
     <kp>1000000.0</kp>
     <kd>100.0</kd>
@@ -79,15 +82,16 @@
       <publishOdomTF>true</publishOdomTF>
       <robotBaseFrame>base_footprint</robotBaseFrame>
+      <robotNameSpace>/</robotNameSpace>
       <publishWheelTF>false</publishWheelTF>
       <publishTf>true</publishTf>
       <publishWheelJointState>true</publishWheelJointState>
       <legacyMode>false</legacyMode>
-      <updateRate>30</updateRate>
+      <updateRate>100</updateRate>
       <leftJoint>wheel_left_joint</leftJoint>
       <rightJoint>wheel_right_joint</rightJoint>
       <wheelSeparation>0.287</wheelSeparation>
       <wheelDiameter>0.066</wheelDiameter>
-      <wheelAcceleration>1</wheelAcceleration>
-      <wheelTorque>10</wheelTorque>
+      <wheelAcceleration>20</wheelAcceleration>
+      <wheelTorque>20</wheelTorque>
       <rosDebugLevel>na</rosDebugLevel>
     </plugin>

File: src/turtlebot3_description/urdf/turtlebot3_waffle.urdf.xacro (robot description, xacro)
@@ -194,5 +194,5 @@
   <parent link="base_link"/>
   <child link="bowl_link"/>
-  <origin rpy="0 0 0" xyz="-0.06 -0.0  0.14"/>
+  <origin rpy="0 0 0" xyz="-0.05 -0.0  0.14"/>
   <axis xyz="0 0 0"/>
 </joint>
@@ -201,5 +201,5 @@
     <origin rpy="0 0 0" xyz="0 0 0"/>
     <geometry>
-      <mesh filename="package://turtlebot3_description/meshes/bowl-version6.stl" scale="0.001 0.001 0.001"/>
+      <mesh filename="package://turtlebot3_description/meshes/bowl-140.stl" scale="0.0030 0.0030 0.0030"/>
     </geometry>
   </visual>
@@ -207,37 +207,41 @@
     <origin rpy="0 0 0" xyz="0 0 0"/>
     <geometry>
-      <mesh filename="package://turtlebot3_description/meshes/bowl-version6.stl" scale="0.001 0.001 0.001"/>
+      <mesh filename="package://turtlebot3_description/meshes/bowl-140.stl" scale="0.0030 0.0030 0.0030"/>
     </geometry>
   </collision>
  <inertial>
-    <mass value="0.01"/>
+    <mass value="0.10"/>
     <origin rpy="0 0 0" xyz="0 0 0"/>
-    <inertia ixx="1" ixy="0" ixz="0" iyy="1" iyz="0" izz="1"/>
+    <inertia ixx="0.1" ixy="0" ixz="0" iyy="0.1" iyz="0" izz="0.2"/>
+    <!--inertia ixx="0.573121008" ixy="4.154e-7" ixz="-2.6e-9" iyy="0.573121008" iyz="7.29e-8" izz="1.0073489184"/-->
+    <!--inertia ixx="5.73121008" ixy="4.154e-6" ixz="-2.6e-8" iyy="5.73121008" iyz="7.29e-7" izz="10.073489184"/-->
+     <!--inertia ixx="0.716401314" ixy="5.1929882325e-7" ixz="-3.242862e-9" iyy="0.716401314" iyz="9.11388915e-8" izz="1.259186148"/-->
   </inertial>
 </link>
-<!--<joint name="ball" type="floating">
+<!--<joint name="base_ball" type="continuous">
+  <origin xyz="0 0 0.2" rpy="0 0 0"/>
   <parent link="base_link"/>
   <child link="ball_link"/>
-  <origin rpy="0 0 0" xyz="0 0 0.3"/>
-  <axis xyz="0 0 0"/>
-</joint>-->
-<!--<link name="ball_link">
- <visual>
- <origin rpy="0 0 0" xyz="0 0 0"/>
- <geometry>
-  <sphere radius="0.01"/>
-</geometry>
- </visual>
-<collision>
-  <origin rpy="0 0 0" xyz="0 0 0"/>
-  <geometry>
-    <sphere radius="0.01"/>
-  </geometry>
-</collision>
-<inertial>
- <mass value="0.01"/>
-  <origin rpy="0 -0 0" xyz=" 0 -0 0"/>
-  <inertia ixx="0.1" ixy="0" ixz="0" iyy="0.1" iyz="0" izz="0.1"/>
-</inertial>
+</joint>
+<link name="ball_link">
+     <visual>
+      <origin xyz="0 0 0" rpy="0.0 -0.0 0.0"/>
+      <geometry>
+            <sphere radius="0.015"/>
+      </geometry>
+    </visual>
+    <collision>
+      <origin xyz="0 0 0" rpy="0 -0 0"/>
+      <geometry>
+            <sphere radius="0.015"/>
+      </geometry>
+    </collision>
+    <inertial>
+      <origin xyz="0 0 0" />
+      <mass value="0.0001" />
+      <inertia ixx="1" ixy="0.0" ixz="0.0"
+               iyy="1" iyz="0.0"
+               izz="1" />
+      </inertial>
 </link>-->
  <!-- <joint name="camera_rgb_joint" type="fixed">
